File: led-power/led-power.kicad_pcb (KiCad board)
At the start: 2 copper layers, 86.4 x 86.4 mm, 70 parts, among them J1 String1, J10 PowerInput, J2 String2, J3 String3, J4 String4, J5 String5, J6 String6, J7 String7, J8 String8, J9 PowerInput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

Commit message: Rev0 of boards; added text
Other:
- board text added: "JLCJLCJLCJLC"
- board text added: "http://github.com/jkominek/piano-conversion LED Power - Rev 0"
Changed lines of the file:
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@@
   (general
     (thickness 1.6)
-    (drawings 32)
+    (drawings 34)
     (tracks 737)
     (zones 0)
@@
   )
   (setup
-    (last_trace_width 1.5)
+    (last_trace_width 0.25)
     (user_trace_width 0.75)
     (user_trace_width 1.5)
@@
       (outputformat 1)
       (mirror false)
-      (drillshape 1)
+      (drillshape 0)
       (scaleselection 1)
-      (outputdirectory ""))
+      (outputdirectory "C:/Users/Jay Kominek/Dropbox/Piano Conversion/x/"))
   )
   (net 0 "")
@@
     )
   )
+  (gr_text JLCJLCJLCJLC (at 78.74 147.32 315) (layer F.SilkS)
+    (effects (font (size 1 1) (thickness 0.15)))
+  )
+  (gr_text "http://github.com/jkominek/piano-conversion\nLED Power - Rev 0" (at 112.776 136.144) (layer F.SilkS)
+    (effects (font (size 1.25 1.25) (thickness 0.2)))
+  )
   (gr_text "NO PROTECTION FROM\nREVERSE POLARITY" (at 111.76 141.986) (layer F.SilkS)
