File: adc-board/ADC Board.sch (KiCad schematic (older format))
At the start: 62 parts, among them J2 ST-LINK/V2, J3 USART3, J4 USART1, J5 UE27AC5410H, J7 AltPowerInput, J8 USBPowerJumper, J9 USART2, U0 STM32H743ZITx, U10 MCP1501-20E/SN, U13 3.3V Reg, U9 USBLC6-2SC6, Y1 NX3225GD-8.000M-EXS00A-CG04874

Commit message: Various changes from initial stages of board bringup
* Add thermal relief to lots of connections
* +3.3V power LED
* BOOT0 jumper for pull to +3.3V
* Reorder USB TVS & ferrite bead
* Tweaking and compaction of some traces
Parts:
- added D5: LED, LEDs:LED_0805_HandSoldering, symbol Device:LED
- added J10: BootJumper, Pin_Headers:Pin_Header_Straight_1x02_Pitch2.54mm, symbol Connector:Conn_01x02_Male
- added R25: CL, Resistors_SMD:R_0805, symbol Device:R_Small_US
Connections:
- net +3V3: now also D5.2 (A), J10.2 (Pin_2)
- net BOOT0: now also J10.1 (Pin_1)
- net GNDD: now also R25.2
- net USB_VBUS: no longer U9.5 (VBUS)
- net at FB1.2, J5.1 (VBUS): now also U9.5 (VBUS)
- new net: D5.1 (K), R25.1
Other:
- moved on the sheet: FB1, J8, R30
Changed lines of the file:
@@
 L power:GNDD #PWR0107
 U 1 1 5F9B2A89
-P 3150 2700
-F 0 "#PWR0107" H 3150 2450 50  0001 C CNN
-F 1 "GNDD" H 3154 2545 50  0000 C CNN
-F 2 "" H 3150 2700 50  0001 C CNN
-F 3 "" H 3150 2700 50  0001 C CNN
-	1    3150 2700
+P 750 3300
+F 0 "#PWR0107" H 750 3050 50  0001 C CNN
+F 1 "GNDD" H 754 3145 50  0000 C CNN
+F 2 "" H 750 3300 50  0001 C CNN
+F 3 "" H 750 3300 50  0001 C CNN
+	1    750  3300
 	1    0    0    -1
 $EndComp
@@
 U 1 1 62BFF5D3
 P 12500 5300
-F 0 "J5" H 12500 6150 50  0000 C CNN
+F 0 "J5" H 12500 5750 50  0000 C CNN
 F 1 "UE27AC5410H" H 12450 5650 50  0000 C CNN
 F 2 "usbconnectors:USB_A_Molex_67643_Horizontal" H 12650 5250 50  0001 C CNN
@@
 L Device:R_Small_US R30
 U 1 1 639EF198
-P 3400 2650
-F 0 "R30" V 3195 2650 50  0000 C CNN
-F 1 "10k" V 3286 2650 50  0000 C CNN
-F 2 "Resistors_SMD:R_0805" H 3400 2650 50  0001 C CNN
-F 3 "~" H 3400 2650 50  0001 C CNN
-	1    3400 2650
+P 1000 3250
+F 0 "R30" V 795 3250 50  0000 C CNN
+F 1 "10k" V 886 3250 50  0000 C CNN
+F 2 "Resistors_SMD:R_0805" H 1000 3250 50  0001 C CNN
+F 3 "~" H 1000 3250 50  0001 C CNN
+	1    1000 3250
 	0    1    1    0
 $EndComp
@@
 	3500 2650 3850 2650
 Wire Wire Line
-	3300 2650 3150 2650
-Wire Wire Line
-	3150 2650 3150 2700
+	900  3250 750  3250
+Wire Wire Line
+	750  3250 750  3300
 Wire Wire Line
 	6350 3150 7050 3150
@@
 L Connector:Conn_01x02_Male J8
 U 1 1 5FC44C17
-P 12550 4500
-F 0 "J8" V 12612 4544 50  0000 L CNN
-F 1 "USBPowerJumper" V 12703 4544 50  0000 L CNN
-F 2 "Pin_Headers:Pin_Header_Straight_1x02_Pitch2.54mm" H 12550 4500 50  0001 C CNN
-F 3 "~" H 12550 4500 50  0001 C CNN
-	1    12550 4500
-	0    1    1    0
-$EndComp
-Wire Wire Line
-	13150 5100 13150 4750
-Wire Wire Line
-	13150 4750 12550 4750
-Wire Wire Line
-	12550 4750 12550 4700
-Wire Wire Line
-	12450 4700 12450 4750
+P 15550 4450
+F 0 "J8" H 15550 4250 50  0000 L CNN
+F 1 "USBPowerJumper" H 15100 4550 50  0000 L CNN
+F 2 "Pin_Headers:Pin_Header_Straight_1x02_Pitch2.54mm" H 15550 4450 50  0001 C CNN
+F 3 "~" H 15550 4450 50  0001 C CNN
+	1    15550 4450
+	-1   0    0    1
+$EndComp
+Wire Wire Line
+	15300 5050 15300 4450
+Wire Wire Line
+	15300 4450 15350 4450
+Wire Wire Line
+	15350 4350 15300 4350
 $Comp
 L power:+5V #PWR0143
 U 1 1 5FC885B1
-P 12250 4700
-F 0 "#PWR0143" H 12250 4550 50  0001 C CNN
-F 1 "+5V" H 12265 4873 50  0000 C CNN
-F 2 "" H 12250 4700 50  0001 C CNN
-F 3 "" H 12250 4700 50  0001 C CNN
-	1    12250 4700
-	1    0    0    -1
-$EndComp
-Wire Wire Line
-	12250 4700 12250 4750
-Wire Wire Line
-	12250 4750 12450 4750
+P 15300 4150
+F 0 "#PWR0143" H 15300 4000 50  0001 C CNN
+F 1 "+5V" H 15315 4323 50  0000 C CNN
+F 2 "" H 15300 4150 50  0001 C CNN
+F 3 "" H 15300 4150 50  0001 C CNN
+	1    15300 4150
+	1    0    0    -1
+$EndComp
+Wire Wire Line
+	15300 4150 15300 4350
 $Comp
 L Device:C C1
@@
 Wire Wire Line
 	12800 5400 13700 5400
-Connection ~ 13150 5100
-Text Label 13550 5100 2    50   ~ 0
-USB_VBUS
 Wire Wire Line
 	6350 3250 8300 3250
@@
 L Device:Ferrite_Bead_Small FB1
 U 1 1 5FC76527
-P 12950 5100
-F 0 "FB1" V 12713 5100 50  0000 C CNN
-F 1 "MPZ2012S601AT000" V 12800 5400 50  0000 C CNN
-F 2 "Inductors_SMD:L_0805" V 12880 5100 50  0001 C CNN
-F 3 "~" H 12950 5100 50  0001 C CNN
-	1    12950 5100
+P 15200 5050
+F 0 "FB1" V 14963 5050 50  0000 C CNN
+F 1 "MPZ2012S601AT000" V 15050 5350 50  0000 C CNN
+F 2 "Inductors_SMD:L_0805" V 15130 5050 50  0001 C CNN
+F 3 "~" H 15200 5050 50  0001 C CNN
+	1    15200 5050
 	0    1    1    0
 $EndComp
@@
 	13600 4650 15100 4650
 Wire Wire Line
-	15100 4650 15100 5350
+	15100 4650 15100 5050
 Wire Wire Line
 	15100 5350 14650 5350
-Wire Wire Line
-	13150 5100 13600 5100
 Text Notes 8400 3300 0    50   ~ 0
 when power is off, PA9 can't exceed 4V.\nthis brings a 5.25V VBUS down to 3.47V.
-Wire Wire Line
-	12800 5100 12850 5100
-Wire Wire Line
-	13050 5100 13150 5100
-$Comp
-L power:+3.3VA #PWR?
+$Comp
+L power:+3.3VA #PWR0126
 U 1 1 5FBE27C1
 P 11400 7000
-F 0 "#PWR?" H 11400 6850 50  0001 C CNN
+F 0 "#PWR0126" H 11400 6850 50  0001 C CNN
 F 1 "+3.3VA" H 11415 7173 50  0000 C CNN
 F 2 "" H 11400 7000 50  0001 C CNN
@@
 $EndComp
 $Comp
-L power:+3.3V #PWR?
+L power:+3.3V #PWR0147
 U 1 1 5FBC7EC8
 P 10750 4600
-F 0 "#PWR?" H 10750 4450 50  0001 C CNN
+F 0 "#PWR0147" H 10750 4450 50  0001 C CNN
 F 1 "+3.3V" H 10765 4773 50  0000 C CNN
 F 2 "" H 10750 4600 50  0001 C CNN
@@
 Wire Wire Line
 	10750 4600 10750 4800
+$Comp
+L Device:LED D5
+U 1 1 5FC9A550
+P 10750 2100
+F 0 "D5" V 10789 1982 50  0000 R CNN
+F 1 "LED" V 10698 1982 50  0000 R CNN
+F 2 "LEDs:LED_0805_HandSoldering" H 10750 2100 50  0001 C CNN
+F 3 "~" H 10750 2100 50  0001 C CNN
+	1    10750 2100
+	0    -1   -1   0
+$EndComp
+$Comp
+L Device:R_Small_US R25
+U 1 1 5FC9A556
+P 10750 2500
+F 0 "R25" H 10818 2546 50  0000 L CNN
+F 1 "CL" H 10818 2455 50  0000 L CNN
+F 2 "Resistors_SMD:R_0805" H 10750 2500 50  0001 C CNN
+F 3 "~" H 10750 2500 50  0001 C CNN
+	1    10750 2500
+	1    0    0    -1
+$EndComp
+Wire Wire Line
+	10750 2400 10750 2250
+Wire Wire Line
+	10750 2600 10750 2650
+Wire Wire Line
+	10750 2650 11500 2650
+Wire Wire Line
+	10750 1950 10750 1850
+$Comp
+L power:+3.3V #PWR0148
+U 1 1 5FD21FA2
+P 10750 1850
+F 0 "#PWR0148" H 10750 1700 50  0001 C CNN
+F 1 "+3.3V" H 10765 2023 50  0000 C CNN
+F 2 "" H 10750 1850 50  0001 C CNN
+F 3 "" H 10750 1850 50  0001 C CNN
+	1    10750 1850
+	1    0    0    -1
+$EndComp
+Wire Wire Line
+	1100 3250 1350 3250
+Text Label 1900 3250 2    50   ~ 0
+BOOT0
+$Comp
+L Connector:Conn_01x02_Male J10
+U 1 1 5FD6D09B
+P 1650 3150
+F 0 "J10" H 1622 3032 50  0000 R CNN
+F 1 "BootJumper" H 1622 3123 50  0000 R CNN
+F 2 "Pin_Headers:Pin_Header_Straight_1x02_Pitch2.54mm" H 1650 3150 50  0001 C CNN
+F 3 "~" H 1650 3150 50  0001 C CNN
+	1    1650 3150
+	-1   0    0    1
+$EndComp
+$Comp
+L power:+3.3V #PWR0149
+U 1 1 5FD6EBC4
+P 1350 2950
+F 0 "#PWR0149" H 1350 2800 50  0001 C CNN
+F 1 "+3.3V" H 1365 3123 50  0000 C CNN
+F 2 "" H 1350 2950 50  0001 C CNN
+F 3 "" H 1350 2950 50  0001 C CNN
+	1    1350 2950
+	1    0    0    -1
+$EndComp
+Wire Wire Line
+	1350 2950 1350 3050
+Wire Wire Line
+	1350 3050 1450 3050
+Wire Wire Line
+	1450 3150 1350 3150
+Wire Wire Line
+	1350 3150 1350 3250
+Connection ~ 1350 3250
+Wire Wire Line
+	1350 3250 1900 3250
+Wire Wire Line
+	12800 5100 13600 5100
+Connection ~ 15100 5050
+Wire Wire Line
+	15100 5050 15100 5350
+Text Label 15300 4700 0    50   ~ 0
+USB_VBUS
 $EndSCHEMATC
