File: adc-board/ADC Board.sch (KiCad schematic (older format))
At the start: 65 parts, among them J10 BootJumper, J2 ST-LINK/V2, J3 USART3, J4 USART1, J5 UE27AC5410H, J7 AltPowerInput, J8 USBPowerJumper, J9 USART2, U0 STM32H743ZITx, U10 MCP1501-20E/SN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

Commit message: Convert analog sensing over to transimpedance amplifiers
Also switched opamps for the TSSOP14 package, and replaced the
fancy voltage reference with a simple 2.0V regulator.
Parts:
- removed C49, C50: 4.3pF, Capacitors_SMD:C_0805, symbol Device:C_Small
- removed C51, C52: 2.2uF, Capacitors_SMD:C_0805, symbol Device:C_Small
- removed R31: 50, Resistors_SMD:R_0805, symbol Device:R_Small_US
- removed U10: MCP1501-20E/SN, SMD_Packages:SOIC-8-N, symbol MCP1501:MCP1501
- removed Y1: NX3225GD-8.000M-EXS00A-CG04874, Crystals:Crystal_SMD_3215-2pin_3.2x1.5mm, symbol Device:Crystal_Small
Connections:
- net Sen10: now also U0.34 (PA0); no longer U0.36 (PA2)
- net Sen12: now also U0.36 (PA2); no longer U0.34 (PA0)
- no-connect marks 69 -> 71
Other:
- note removed: "Don't intend to need this crystal circuit"
- note removed: "Vref will be 2.048V, leaving much headroom between it at VDDA at 3.3V.\nThe resistors need to be chosen to keep (VDDA - R*maxcurrent) >> Vcesat (0.3V).\nR*maxcurrent should also be slightly less than Vref, which has to be chosen from\navailable voltage reference parts."
- moved on the sheet: C53, C54, C55, C56, JP0, U13

Commit message: convert to surface mount caps for power filtration
Parts:
- C53: footprint Capacitors_THT:CP_Radial_D5.0mm_P2.00mm -> Capacitors_SMD:CP_Elec_4x4.5
- C54: footprint Capacitors_THT:CP_Radial_D6.3mm_P2.50mm -> Capacitors_SMD:CP_Elec_5x5.3
Changed lines of the file:
@@
 F 0 "C53" H 11891 7746 50  0000 L CNN
 F 1 "10uF EEA-GA1V100" H 11891 7655 50  0000 L CNN
-F 2 "Capacitors_THT:CP_Radial_D5.0mm_P2.00mm" H 11800 7700 50  0001 C CNN
+F 2 "Capacitors_SMD:CP_Elec_4x4.5" H 11800 7700 50  0001 C CNN
 F 3 "~" H 11800 7700 50  0001 C CNN
 	1    11800 7700
@@
 F 0 "C54" H 12691 7746 50  0000 L CNN
 F 1 "22uF ECE-A1HKA220" H 12691 7655 50  0000 L CNN
-F 2 "Capacitors_THT:CP_Radial_D6.3mm_P2.50mm" H 12600 7700 50  0001 C CNN
+F 2 "Capacitors_SMD:CP_Elec_5x5.3" H 12600 7700 50  0001 C CNN
 F 3 "~" H 12600 7700 50  0001 C CNN
 	1    12600 7700

Commit message: Fix swapped RS485 Z/Y pins. Add reset supervisor and 4 pin USB header.
Parts:
- added J11: USB Header, Pin_Headers:Pin_Header_Straight_1x04_Pitch2.54mm, symbol Connector:Conn_01x04_Male
- added U7: MCP120-xxxxTT, TO_SOT_Packages_SMD:SOT-23, symbol Power_Supervisor:MCP120-xxxxTT
Connections:
- net +3V3: now also U7.2 (VDD)
- net GNDD: now also J11.1 (Pin_1), U7.3 (VSS)
- net NRST: now also U7.1 (~RST)
- net USB_D+: now also J11.2 (Pin_2)
- net USB_D-: now also J11.3 (Pin_3)
- net at FB1.2, J5.1 (VBUS), U9.5 (VBUS): now also J11.4 (Pin_4)
Other:
- moved on the sheet: J10, R30
Changed lines of the file:
@@
 L power:GNDD #PWR0107
 U 1 1 5F9B2A89
-P 750 3300
-F 0 "#PWR0107" H 750 3050 50  0001 C CNN
-F 1 "GNDD" H 754 3145 50  0000 C CNN
-F 2 "" H 750 3300 50  0001 C CNN
-F 3 "" H 750 3300 50  0001 C CNN
-	1    750  3300
+P 1950 4250
+F 0 "#PWR0107" H 1950 4000 50  0001 C CNN
+F 1 "GNDD" H 1954 4095 50  0000 C CNN
+F 2 "" H 1950 4250 50  0001 C CNN
+F 3 "" H 1950 4250 50  0001 C CNN
+	1    1950 4250
 	1    0    0    -1
 $EndComp
@@
 L Device:R_Small_US R30
 U 1 1 639EF198
-P 1000 3250
-F 0 "R30" V 795 3250 50  0000 C CNN
-F 1 "10k" V 886 3250 50  0000 C CNN
-F 2 "Resistors_SMD:R_0805" H 1000 3250 50  0001 C CNN
-F 3 "~" H 1000 3250 50  0001 C CNN
-	1    1000 3250
+P 2200 4200
+F 0 "R30" V 1995 4200 50  0000 C CNN
+F 1 "10k" V 2086 4200 50  0000 C CNN
+F 2 "Resistors_SMD:R_0805" H 2200 4200 50  0001 C CNN
+F 3 "~" H 2200 4200 50  0001 C CNN
+	1    2200 4200
 	0    1    1    0
 $EndComp
@@
 	3500 2650 3850 2650
 Wire Wire Line
-	900  3250 750  3250
-Wire Wire Line
-	750  3250 750  3300
+	2100 4200 1950 4200
+Wire Wire Line
+	1950 4200 1950 4250
 Wire Wire Line
 	6350 3150 7050 3150
@@
 $EndComp
 Wire Wire Line
-	2150 2650 2150 2700
+	2150 2650 2150 2800
 $Comp
 L power:GNDD #PWR0144
 U 1 1 5FD3C9A6
-P 2150 2700
-F 0 "#PWR0144" H 2150 2450 50  0001 C CNN
-F 1 "GNDD" H 2154 2545 50  0000 C CNN
-F 2 "" H 2150 2700 50  0001 C CNN
-F 3 "" H 2150 2700 50  0001 C CNN
-	1    2150 2700
-	1    0    0    -1
-$EndComp
-Wire Wire Line
-	12800 5300 13700 5300
-Wire Wire Line
-	12800 5400 13700 5400
+P 2150 2900
+F 0 "#PWR0144" H 2150 2650 50  0001 C CNN
+F 1 "GNDD" H 2154 2745 50  0000 C CNN
+F 2 "" H 2150 2900 50  0001 C CNN
+F 3 "" H 2150 2900 50  0001 C CNN
+	1    2150 2900
+	1    0    0    -1
+$EndComp
+Wire Wire Line
+	12800 5300 13000 5300
+Wire Wire Line
+	12800 5400 12950 5400
 Wire Wire Line
 	6350 3250 8300 3250
@@
 $EndComp
 Wire Wire Line
-	1100 3250 1350 3250
-Text Label 1900 3250 2    50   ~ 0
+	2300 4200 2550 4200
+Text Label 3100 4200 2    50   ~ 0
 BOOT0
 $Comp
 L Connector:Conn_01x02_Male J10
 U 1 1 5FD6D09B
-P 1650 3150
-F 0 "J10" H 1622 3032 50  0000 R CNN
-F 1 "BootJumper" H 1622 3123 50  0000 R CNN
-F 2 "Pin_Headers:Pin_Header_Straight_1x02_Pitch2.54mm" H 1650 3150 50  0001 C CNN
-F 3 "~" H 1650 3150 50  0001 C CNN
-	1    1650 3150
+P 2850 4100
+F 0 "J10" H 2822 3982 50  0000 R CNN
+F 1 "BootJumper" H 2822 4073 50  0000 R CNN
+F 2 "Pin_Headers:Pin_Header_Straight_1x02_Pitch2.54mm" H 2850 4100 50  0001 C CNN
+F 3 "~" H 2850 4100 50  0001 C CNN
+	1    2850 4100
 	-1   0    0    1
 $EndComp
@@
 L power:+3.3V #PWR0149
 U 1 1 5FD6EBC4
-P 1350 2950
-F 0 "#PWR0149" H 1350 2800 50  0001 C CNN
-F 1 "+3.3V" H 1365 3123 50  0000 C CNN
-F 2 "" H 1350 2950 50  0001 C CNN
-F 3 "" H 1350 2950 50  0001 C CNN
-	1    1350 2950
-	1    0    0    -1
-$EndComp
-Wire Wire Line
-	1350 2950 1350 3050
-Wire Wire Line
-	1350 3050 1450 3050
-Wire Wire Line
-	1450 3150 1350 3150
-Wire Wire Line
-	1350 3150 1350 3250
-Connection ~ 1350 3250
-Wire Wire Line
-	1350 3250 1900 3250
-Wire Wire Line
-	12800 5100 13600 5100
+P 2550 3900
+F 0 "#PWR0149" H 2550 3750 50  0001 C CNN
+F 1 "+3.3V" H 2565 4073 50  0000 C CNN
+F 2 "" H 2550 3900 50  0001 C CNN
+F 3 "" H 2550 3900 50  0001 C CNN
+	1    2550 3900
+	1    0    0    -1
+$EndComp
+Wire Wire Line
+	2550 3900 2550 4000
+Wire Wire Line
+	2550 4000 2650 4000
+Wire Wire Line
+	2650 4100 2550 4100
+Wire Wire Line
+	2550 4100 2550 4200
+Connection ~ 2550 4200
+Wire Wire Line
+	2550 4200 3100 4200
+Wire Wire Line
+	12800 5100 13050 5100
 Connection ~ 15100 5050
 Wire Wire Line
@@
 NoConn ~ 3850 3750
 NoConn ~ 3850 3850
+$Comp
+L Power_Supervisor:MCP120-xxxxTT U7
+U 1 1 61F80A9F
+P 1700 2350
+F 0 "U7" H 1470 2396 50  0000 R CNN
+F 1 "MCP120-xxxxTT" H 1470 2305 50  0000 R CNN
+F 2 "TO_SOT_Packages_SMD:SOT-23" H 2300 2000 50  0001 C CNN
+F 3 "http://ww1.microchip.com/downloads/en/DeviceDoc/11184d.pdf" H 1700 2350 50  0001 C CNN
+	1    1700 2350
+	1    0    0    -1
+$EndComp
+Wire Wire Line
+	3650 1900 1700 1900
+Wire Wire Line
+	1700 1900 1700 1950
+Connection ~ 3650 1900
+Wire Wire Line
+	1700 2750 1700 2800
+Wire Wire Line
+	1700 2800 2150 2800
+Connection ~ 2150 2800
+Wire Wire Line
+	2150 2800 2150 2900
+Wire Wire Line
+	2000 2350 2150 2350
+Connection ~ 2150 2350
+$Comp
+L Connector:Conn_01x04_Male J11
+U 1 1 6201C3CD
+P 13300 6000
+F 0 "J11" H 13272 5882 50  0000 R CNN
+F 1 "USB Header" H 13272 5973 50  0000 R CNN
+F 2 "Pin_Headers:Pin_Header_Straight_1x04_Pitch2.54mm" H 13300 6000 50  0001 C CNN
+F 3 "~" H 13300 6000 50  0001 C CNN
+	1    13300 6000
+	-1   0    0    1
+$EndComp
+Wire Wire Line
+	13100 5800 13050 5800
+Wire Wire Line
+	13050 5800 13050 5100
+Connection ~ 13050 5100
+Wire Wire Line
+	13050 5100 13600 5100
+Wire Wire Line
+	13000 5300 13000 6000
+Connection ~ 13000 5300
+Wire Wire Line
+	13000 5300 13700 5300
+Wire Wire Line
+	12950 5400 12950 5900
+Connection ~ 12950 5400
+Wire Wire Line
+	12950 5400 13700 5400
+Wire Wire Line
+	13100 6100 12900 6100
+Wire Wire Line
+	12900 6100 12900 5750
+Wire Wire Line
+	12900 5750 12500 5750
+Wire Wire Line
+	12950 5900 13100 5900
+Wire Wire Line
+	13000 6000 13100 6000
 $EndSCHEMATC

Commit message: Swap USART1 and USART3 on RS485 connection, so that main board has bootloader access.
Parts:
- J4: footprint Pin_Headers:Pin_Header_Straight_1x03_Pitch1.27mm -> Pin_Headers:Pin_Header_Straight_1x03_Pitch2.54mm
Changed lines of the file:
@@
 F 0 "J4" H 13258 4331 50  0000 C CNN
 F 1 "USART1" H 13258 4240 50  0000 C CNN
-F 2 "Pin_Headers:Pin_Header_Straight_1x03_Pitch1.27mm" H 13150 4050 50  0001 C CNN
+F 2 "Pin_Headers:Pin_Header_Straight_1x03_Pitch2.54mm" H 13150 4050 50  0001 C CNN
 F 3 "~" H 13150 4050 50  0001 C CNN
 	1    13150 4050
@@
 	11950 3800 11400 3800
 Text Label 11400 3600 0    50   ~ 0
-USART1_RX
+USART3_RX
 Text Label 11400 3800 0    50   ~ 0
-USART1_TX
+USART3_TX
 $Comp
 L Device:LED D1

Commit message: First batch of ADC rev 2 changes
* Pulled JTAG header in from the edge
* External power header silkscreen
* Increased most thermal relief
* Relocated 3.3V power indicator LED
* Increased electrolytic cap footprint
Parts:
- C53: footprint Capacitors_SMD:CP_Elec_4x4.5 -> Capacitors_SMD:CP_Elec_5x5.3
- C54: footprint Capacitors_SMD:CP_Elec_5x5.3 -> Capacitors_SMD:CP_Elec_6.3x5.3
- H1, H2, H3, H4: footprint Mounting_Holes:MountingHole_3.2mm_M3_Pad -> Mounting_Holes:MountingHole_3.2mm_M3_Pad_Via
Changed lines of the file:
@@
 F 0 "H1" H 1100 1399 50  0000 L CNN
 F 1 "MountingHole_Pad" H 1100 1308 50  0000 L CNN
-F 2 "Mounting_Holes:MountingHole_3.2mm_M3_Pad" H 1000 1350 50  0001 C CNN
+F 2 "Mounting_Holes:MountingHole_3.2mm_M3_Pad_Via" H 1000 1350 50  0001 C CNN
 F 3 "~" H 1000 1350 50  0001 C CNN
 	1    1000 1350
@@
 F 0 "H2" H 1400 1399 50  0000 L CNN
 F 1 "MountingHole_Pad" H 1400 1308 50  0000 L CNN
-F 2 "Mounting_Holes:MountingHole_3.2mm_M3_Pad" H 1300 1350 50  0001 C CNN
+F 2 "Mounting_Holes:MountingHole_3.2mm_M3_Pad_Via" H 1300 1350 50  0001 C CNN
 F 3 "~" H 1300 1350 50  0001 C CNN
 	1    1300 1350
@@
 F 0 "H3" H 1700 1399 50  0000 L CNN
 F 1 "MountingHole_Pad" H 1700 1308 50  0000 L CNN
-F 2 "Mounting_Holes:MountingHole_3.2mm_M3_Pad" H 1600 1350 50  0001 C CNN
+F 2 "Mounting_Holes:MountingHole_3.2mm_M3_Pad_Via" H 1600 1350 50  0001 C CNN
 F 3 "~" H 1600 1350 50  0001 C CNN
 	1    1600 1350
@@
 F 0 "H4" H 2000 1399 50  0000 L CNN
 F 1 "MountingHole_Pad" H 2000 1308 50  0000 L CNN
-F 2 "Mounting_Holes:MountingHole_3.2mm_M3_Pad" H 1900 1350 50  0001 C CNN
+F 2 "Mounting_Holes:MountingHole_3.2mm_M3_Pad_Via" H 1900 1350 50  0001 C CNN
 F 3 "~" H 1900 1350 50  0001 C CNN
 	1    1900 1350
@@
 F 0 "C53" H 11891 7746 50  0000 L CNN
 F 1 "10uF EEA-GA1V100" H 11891 7655 50  0000 L CNN
-F 2 "Capacitors_SMD:CP_Elec_4x4.5" H 11800 7700 50  0001 C CNN
+F 2 "Capacitors_SMD:CP_Elec_5x5.3" H 11800 7700 50  0001 C CNN
 F 3 "~" H 11800 7700 50  0001 C CNN
 	1    11800 7700
@@
 F 0 "C54" H 12691 7746 50  0000 L CNN
 F 1 "22uF ECE-A1HKA220" H 12691 7655 50  0000 L CNN
-F 2 "Capacitors_SMD:CP_Elec_5x5.3" H 12600 7700 50  0001 C CNN
+F 2 "Capacitors_SMD:CP_Elec_6.3x5.3" H 12600 7700 50  0001 C CNN
 F 3 "~" H 12600 7700 50  0001 C CNN
 	1    12600 7700
