File: link-adapter/link-adapter.kicad_pcb (KiCad board)
At the start: 2 copper layers, 77.5 x 40.6 mm, 41 parts, among them J1 ToADC, J2 ToMaster, J3 USB_B, J4 FTDI Header, J5 PowerJumper, J6 CBUS, J7 FORLED, J8 AltUSB, Q1 NX7002BKW, U1 ISL83490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

Commit message: include GND in power jumper header so it can receive external power
Parts:
- J5: footprint Pin_Headers:Pin_Header_Straight_1x02_Pitch2.54mm -> Pin_Headers:Pin_Header_Straight_1x04_Pitch2.54mm
- moved J5 5.80 mm to (117.1, 76.7)

Commit message: Rev0 of boards; added text
Other:
- board text added: "http://github.com/jkominek/piano-conversion Link Adapter - Rev 0"

Commit message: fix missing ground in rev0; adjust silk screen for readability
Routing:
- net GND: track 48.9 -> 55.5 mm

Commit message: Add a header for measuring current to ADC board
Parts:
- added J9: CurrentProbe, Pin_Headers:Pin_Header_Straight_1x02_Pitch2.54mm, F.Cu at (136.7, 78.0)
- R11: value 1500 -> 620
Connections:
- C8 pad 1: +5V -> Net-(C8-Pad1)
- J1 pad 3: +5V -> Net-(C8-Pad1)
- J1 pad 5: +5V -> Net-(C8-Pad1)
Routing:
- net Net-(C8-Pad1): track 0.00 -> 32.0 mm
- net +5V: track 56.6 -> 29.5 mm
Other:
- board text added: "CurrentProbe"

Commit message: Silkscreen improvements for usability
Connections:
- net Net-(J6-Pad1) renamed /CBUS1
- net Net-(J6-Pad2) renamed /CBUS3
- net Net-(J6-Pad3) renamed /CBUS0
- net Net-(J6-Pad4) renamed /CBUS2
Other:
- board text added: "+3.3V"
- board text added: "0"
- board text added: "1"
- board text added: "2"
- board text added: "3"
- board text added: "5V"
- board text added: "D+"
- board text added: "D-"
- board text added: "FTDI RX"
- board text added: "FTDI TX"
- board text added: "GND"
- board text added: "NC"

Commit message: Add/update board rev silkscreen, nothing else
Other:
- board text added: "http://github.com/jkominek/piano-conversion Link Adapter - Rev 1"
- board text removed: "http://github.com/jkominek/piano-conversion Link Adapter - Rev 0"
