File: sensorboards/2040-centered-1x/2040-centered-1x.kicad_pcb (KiCad board)
At the start: 2 copper layers, 8 x 48 mm, 8 parts, among them J1 Conn_02x02_Odd_Even, U1 CNY70

Commit message: Made issue #44 changes to sensorboards, introduced 3x versions
Also finished bringing them up to Kicad 6.0
Parts:
- moved H2 0.08 mm to (175.0, 110.0)
- moved H1 0.07 mm to (175.0, 130.0)
Routing:
- net /Anode: track 24.2 -> 33.2 mm, vias 1 -> 0
- net /Cathode: track 24.2 -> 33.0 mm
- net /Collector: track 33.3 -> 37.7 mm
- net /Emitter: track 33.2 -> 34.4 mm
Other:
- net class Default removed
