File: hardware/midi-board/midi-board.kicad_sch (KiCad schematic)
At the start: 37 parts, among them J1 MIDI OUT, J10 Conn_02x02_Odd_Even, J2 MIDI IN, J3 Qwiic, J4 Serial Wire, J6 Qwiic, J7 UART, J8 I2C, Q1 Q_NPN_BEC, Q2 Q_NPN_BEC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

Commit message: Convert all other mounting holes to non-pad variety.
Reroute a few traces to be shorter.
Parts:
- H1, H2, H3: footprint Mounting_Holes:MountingHole_3.2mm_M3_Pad_Via -> MountingHole:MountingHole_3.2mm_M3
