File: hardware/main-board/Power.kicad_sch (KiCad schematic)
At the start: 55 parts, among them J4 5V Input, Q1 N Channel, Q10 N Channel, Q11 N Channel, Q12 N Channel, Q13 P Channel, Q14 P Channel, Q15 P Channel, Q16 P Channel, Q17 P Channel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

Commit message: Next revs of the important boards
Includes some tiny DRC tweaks for the LED power board.
Connections:
- net PWR2_PG: now reaches Q1.3 (D), Q5.1 (G), R24.2
- net PWR4_PG: now reaches Q13.1 (G), Q9.3 (D), R36.2
- net PWR3_PG: now reaches Q2.3 (D), Q6.1 (G), R26.2
- net PWR1_PG: now reaches Q10.3 (D), Q14.1 (G), R38.2
- net PWR5_PG: now reaches Q3.3 (D), Q7.1 (G), R28.2
- net PWR7_PG: now reaches Q11.3 (D), Q15.1 (G), R40.2
- net PWR8_PG: now reaches Q4.3 (D), Q8.1 (G), R30.2
- net PWR6_PG: now reaches Q12.3 (D), Q16.1 (G), R42.2
Changed lines of the file:
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@@
     (stroke (width 0) (type default) (color 0 0 0 0))
+  )
+  (label "PWR4_PG" (at 173.99 33.02 180)
+    (effects (font (size 1.27 1.27)) (justify right bottom))
+  )
+  (label "PWR3_PG" (at 118.11 72.39 180)
+    (effects (font (size 1.27 1.27)) (justify right bottom))
+  )
+  (label "PWR2_PG" (at 118.11 33.02 180)
+    (effects (font (size 1.27 1.27)) (justify right bottom))
+  )
+  (label "PWR8_PG" (at 118.11 147.32 180)
+    (effects (font (size 1.27 1.27)) (justify right bottom))
+  )
+  (label "PWR1_PG" (at 173.99 72.39 180)
+    (effects (font (size 1.27 1.27)) (justify right bottom))
+  )
+  (label "PWR5_PG" (at 118.11 110.49 180)
+    (effects (font (size 1.27 1.27)) (justify right bottom))
+  )
+  (label "PWR7_PG" (at 173.99 110.49 180)
+    (effects (font (size 1.27 1.27)) (justify right bottom))
+  )
+  (label "PWR6_PG" (at 173.99 147.32 180)
+    (effects (font (size 1.27 1.27)) (justify right bottom))
   )
   (global_label "PWR4" (shape input) (at 194.31 39.37 0) (fields_autoplaced)
