File: hardware/sensorboards/2040-centered-2x-QRE1113GR/2040-centered-2x.kicad_sch (KiCad schematic)
At the start: 8 parts, among them J1 Conn_01x06_Male, U1 QRE1113GR, U2 QRE1113GR

Commit message: Straight connector Adjusted board size 3D models of parts Raytracing rendering
Parts:
- J1: footprint Pin_Headers:Pin_Header_Angled_1x06_Pitch2.54mm -> Connector_PinHeader_2.54mm:PinHeader_1x06_P2.54mm_Vertical
Changed lines of the file:
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@@
   )
   (symbol (lib_id "Connector:Conn_01x06_Male") (at 100.33 45.72 270) (unit 1)
-    (in_bom yes) (on_board yes)
-    (property "Reference" "J1" (id 0) (at 106.5276 47.2948 90)
-      (effects (font (size 1.27 1.27)) (justify left))
-    )
-    (property "Value" "Conn_01x06_Male" (id 1) (at 106.5276 49.6062 90)
-      (effects (font (size 1.27 1.27)) (justify left))
-    )
-    (property "Footprint" "Pin_Headers:Pin_Header_Angled_1x06_Pitch2.54mm" (id 2) (at 100.33 45.72 0)
+    (in_bom yes) (on_board yes) (fields_autoplaced)
+    (property "Reference" "J1" (id 0) (at 99.06 40.64 90))
+    (property "Value" "Conn_01x06_Male" (id 1) (at 99.06 43.18 90))
+    (property "Footprint" "Connector_PinHeader_2.54mm:PinHeader_1x06_P2.54mm_Vertical" (id 2) (at 100.33 45.72 0)
       (effects (font (size 1.27 1.27)) hide)
     )
@@
       (reference "H4") (unit 1) (value "MountingHole") (footprint "Mounting_Holes:MountingHole_3.2mm_M3")
     )
-    (path "/00000000-0000-0000-0000-0000603b900c"
-      (reference "J1") (unit 1) (value "Conn_01x06_Male") (footprint "Pin_Headers:Pin_Header_Angled_1x06_Pitch2.54mm")
+    (path "/0da2b054-fc0f-44e0-870c-d9652a404c75"
+      (reference "J1") (unit 1) (value "Conn_01x06_Male") (footprint "Connector_PinHeader_2.54mm:PinHeader_1x06_P2.54mm_Vertical")
     )
     (path "/a4ed41dc-eb94-4e3f-a482-d012214b0b8a"
