File: hardware/sensorboards/2040-centered-4x-QRE1113GR/rendering/render.kicad_pcb (KiCad board)
At the start: 2 copper layers, 174.6 x 52 mm, 44 parts, among them J1 Conn_01x10_Male, U1 QRE1113GR, U2 QRE1113GR, U3 QRE1113GR, U4 QRE1113GR

Commit message: new PCB into the old rendering file, what a pain! But at least it works...
Parts:
- removed the H1 at (70.8, 82.3)
- removed the H1 at (196.4, 82.3)
- removed the H1 at (142.1, 82.3)
- removed the H2 at (142.1, 102.3)
- removed the H2 at (70.8, 102.3)
- removed the H2 at (196.4, 102.3)
- removed the H3 at (83.4, 82.3)
- removed the H3 at (154.7, 82.3)
- removed the H3 at (209.0, 82.3)
- removed the H4 at (154.7, 102.3)
- removed the H4 at (209.0, 102.3)
- removed the H4 at (83.4, 102.3)
- removed the H5 at (96.0, 82.3)
- removed the H5 at (221.6, 82.3)
- removed the H5 at (167.3, 82.3)
- removed the H6 at (167.3, 102.3)
- removed the H6 at (221.6, 102.3)
- removed the H6 at (96.0, 102.3)
- removed the J1 at (71.8, 62.4)
- removed the J1 at (220.4, 62.4)
- removed the J1 at (166.1, 62.4)
- removed the TP1 at (63.8, 108.3)
- removed the TP1 at (189.4, 108.3)
- removed the TP1 at (135.1, 108.3)
- removed the TP2 at (148.1, 108.3)
- removed the TP2 at (76.8, 108.3)
- removed the TP2 at (202.4, 108.3)
- removed the TP3 at (174.1, 108.3)
- removed the TP3 at (228.4, 108.3)
- removed the TP3 at (102.8, 108.3)
- removed the U1 at (135.8, 92.3)
- removed the U1 at (64.5, 92.3)
- removed the U1 at (190.1, 92.3)
- removed the U2 at (202.7, 92.3)
- removed the U2 at (77.1, 92.3)
- removed the U2 at (148.4, 92.3)
- removed the U3 at (215.3, 92.3)
- removed the U3 at (161.0, 92.3)
- removed the U3 at (89.7, 92.3)
- removed the U4 at (227.9, 92.3)
- removed the U4 at (173.6, 92.3)
- removed the U4 at (102.3, 92.3)
- added H1: MountingHole, Mounting_Holes:MountingHole_3.2mm_M3, F.Cu at (40.6, 82.3)
- added H1: MountingHole, Mounting_Holes:MountingHole_3.2mm_M3, F.Cu at (141.9, 82.3)
- added H1: MountingHole, Mounting_Holes:MountingHole_3.2mm_M3, F.Cu at (196.3, 81.9)
- added H2: MountingHole, Mounting_Holes:MountingHole_3.2mm_M3, F.Cu at (141.9, 102.3)
- added H2: MountingHole, Mounting_Holes:MountingHole_3.2mm_M3, F.Cu at (40.6, 102.3)
- added H2: MountingHole, Mounting_Holes:MountingHole_3.2mm_M3, F.Cu at (196.3, 101.9)
- added H3: MountingHole, Mounting_Holes:MountingHole_3.2mm_M3, F.Cu at (154.6, 82.3)
- added H3: MountingHole, Mounting_Holes:MountingHole_3.2mm_M3, F.Cu at (208.9, 81.9)
- added H3: MountingHole, Mounting_Holes:MountingHole_3.2mm_M3, F.Cu at (53.2, 82.3)
- added H4: MountingHole, Mounting_Holes:MountingHole_3.2mm_M3, F.Cu at (53.2, 102.3)
- added H4: MountingHole, Mounting_Holes:MountingHole_3.2mm_M3, F.Cu at (208.9, 101.9)
- added H4: MountingHole, Mounting_Holes:MountingHole_3.2mm_M3, F.Cu at (154.6, 102.3)
- added H5: MountingHole, Mounting_Holes:MountingHole_3.2mm_M3, F.Cu at (65.8, 82.3)
- added H5: MountingHole, Mounting_Holes:MountingHole_3.2mm_M3, F.Cu at (167.2, 82.3)
- added H5: MountingHole, Mounting_Holes:MountingHole_3.2mm_M3, F.Cu at (221.6, 81.9)
- added H6: MountingHole, Mounting_Holes:MountingHole_3.2mm_M3, F.Cu at (221.6, 101.9)
- added H6: MountingHole, Mounting_Holes:MountingHole_3.2mm_M3, F.Cu at (167.2, 102.3)
- added H6: MountingHole, Mounting_Holes:MountingHole_3.2mm_M3, F.Cu at (65.8, 102.3)
- added J1: Conn_01x10_Male, Connector_PinHeader_2.54mm:PinHeader_1x10_P2.54mm_Vertical, F.Cu at (41.7, 62.4)
- added J1: Conn_01x10_Male, Connector_PinHeader_2.54mm:PinHeader_1x10_P2.54mm_Vertical, B.Cu at (165.9, 62.4)
- added J1: Conn_01x10_Male, Connector_PinHeader_2.54mm:PinHeader_1x10_P2.54mm_Vertical, B.Cu at (220.3, 62.0)
- added TP1: TestPoint, TestPoint:TestPoint_Pad_1.0x1.0mm, F.Cu at (134.9, 108.3)
- added TP1: TestPoint, TestPoint:TestPoint_Pad_1.0x1.0mm, F.Cu at (189.3, 107.9)
- added TP1: TestPoint, TestPoint:TestPoint_Pad_1.0x1.0mm, F.Cu at (33.6, 108.3)
- added TP2: TestPoint, TestPoint:TestPoint_Pad_1.0x1.0mm, F.Cu at (147.9, 108.3)
- added TP2: TestPoint, TestPoint:TestPoint_Pad_1.0x1.0mm, F.Cu at (202.3, 107.9)
- added TP2: TestPoint, TestPoint:TestPoint_Pad_1.0x1.0mm, F.Cu at (46.6, 108.3)
- added TP3: TestPoint, TestPoint:TestPoint_Pad_1.0x1.0mm, F.Cu at (228.3, 107.9)
- added TP3: TestPoint, TestPoint:TestPoint_Pad_1.0x1.0mm, F.Cu at (72.7, 108.3)
- added TP3: TestPoint, TestPoint:TestPoint_Pad_1.0x1.0mm, F.Cu at (173.9, 108.3)
- added U1: QRE1113GR, OptoDevice:QRE1113GR, F.Cu at (34.4, 92.3)
- added U1: QRE1113GR, OptoDevice:QRE1113GR, F.Cu at (190.1, 91.9)
- added U1: QRE1113GR, OptoDevice:QRE1113GR, F.Cu at (135.7, 92.3)
- added U2: QRE1113GR, OptoDevice:QRE1113GR, F.Cu at (47.0, 92.3)
- added U2: QRE1113GR, OptoDevice:QRE1113GR, F.Cu at (202.7, 91.9)
- added U2: QRE1113GR, OptoDevice:QRE1113GR, F.Cu at (148.2, 92.3)
- added U3: QRE1113GR, OptoDevice:QRE1113GR, F.Cu at (160.8, 92.3)
- added U3: QRE1113GR, OptoDevice:QRE1113GR, F.Cu at (215.2, 91.9)
- added U3: QRE1113GR, OptoDevice:QRE1113GR, F.Cu at (59.5, 92.3)
- added U4: QRE1113GR, OptoDevice:QRE1113GR, F.Cu at (173.4, 92.3)
- added U4: QRE1113GR, OptoDevice:QRE1113GR, F.Cu at (72.2, 92.3)
- added U4: QRE1113GR, OptoDevice:QRE1113GR, F.Cu at (227.8, 91.9)
Other:
- board size 174.6 x 52 mm -> 204.8 x 52 mm
- board text added: "+"
- board text added: "-"
- board text added: "C"
- board text added: "E"
